File: TMK-EURO.sch (EAGLE design)
At the start: 38 parts, among them IC1 TL082P, U1 IN, U2 THONKICONNOLD

Commit message: Final schematic design
breadboard check
Parts:
- removed D7: 1N1004, MusicThingModular:SMALL_DIODEDO35-7
- added C1: 1uF, rcl:C-EU050-035X075
- added C11, C4: 100nF, rcl:C-EU050-035X075
- added OK1, OK2: 4N35, optocoupler:4N35
- added OUTPUT1, OUTPUT2, U3, U4, U6: IN, MusicThingModular:THONKICONNOLD
- added R10, R8: 5K6, adafruit:R-US_0207/7
- added R11, R9: 3K3, adafruit:R-US_0207/7
- added R14: 100k, adafruit:R-US_0207/7
- added R15: 47k, adafruit:R-US_0207/7
- added R16: 10K, adafruit:R-US_0207/7
- added S1: (no value), switch:320-916
- added VR16: 1k, MusicThingModular:9MM_SNAP-IN_POT_
- C10: value 100nF -> 220pF; device adafruit:C-US050-030X075 -> rcl:C-EU050-035X075
- C2, C3, C5, C9: value 1uF -> 100nF; device adafruit:C-US050-030X075 -> rcl:C-EU050-035X075
- C6: value 2uF -> 2.2uF
- D2: value 1N1004 -> 1N5817
- LED1, LED2: value RED -> oranger
- VR13: value 100K -> 250K
- VR14: value 100K -> 500k
Connections:
- new net BYPASS: S1.P, VR7.A
- new net N$23: R6.1, VR16.S
- new net N$27: OK1.EMI, R9.2
- new net N$28: OK1.C, R8.1
- new net N$29: R15.1, VR14.A
- new net N$30: OK1.A, U3.TIP
- new net N$31: OK2.EMI, R11.1
- new net N$32: OK2.C, R10.1
- new net N$33: OK2.A, U4.TIP
- new net N$34: S1.S
- new net N$35: C9.2, OUTPUT2.TIP
- new net N$36: C11.1, R16.2
- new net N$40: C11.2, U6.SLEEVE
- new net OUTPUT1: C4.1, VR13.E, VR13.S
- new net OUTPUT2: C10.2, C9.1, VR14.E, VR14.S
- net +12V: now also VR16.E; no longer R6.1
- net GND: now also C10.1, OUTPUT1.SLEEVE, OUTPUT2.SLEEVE, R10.2, R8.2, U3.SLEEVE, U4.SLEEVE, VR16.A; no longer C10.2, D7.C
- net N$10: now also R14.2
- net N$13: now also R15.2
- net N$18: now also C1.1; no longer C9.1
- net N$2: now also OK2.COL
- net N$20: now also C1.2; no longer C9.2, VR13.E, VR14.E
- net N$25: now also C4.2, OUTPUT1.TIP; no longer D7.A, VR13.A, VR13.S
- net N$26: now also R14.1, VR13.A; no longer C10.1, VR14.A, VR14.S
- net N$4: now also OK1.COL
- net N$5: now also R16.1, R9.1
- net N$7: now also S1.O; no longer VR7.A
- net N$9: now also R11.2
Other:
- note added: "BIASPEAK"
- note added: "LEDcomp"
- note added: "bias"
- note added: "bypass"
- note added: "feedbackgain"
- note added: "freq modulation"
- note added: "leakback"
- note added: "level"
- note added: "mufflepass"
- note added: "outlvl"
- note added: "output stage 1"
- note added: "output stage 2"
- note added: "output2"
- note added: "resonator"
- note added: "starvere"
- note added: "switch"
- moved on the sheet: C10, C7, C8, C9, D2, R3, R6, R7, U1, VR1, VR13, VR14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
