File: TMK-EURO-0.1.1.brd (EAGLE design)
At the start: 100 x 80 mm, 56 parts, among them IC1 TL082P, U1 IN, U2 IN, U3 IN, U4 IN, U5 IN, U6 IN, U7 THONKICONNOLD

Commit message: final design frontpanel include
Parts:
- C11: device rcl:C050-035X075 -> adafruit:C050-075X075
- moved C11 1.27 mm to (55.9, 76.2)
Routing:
- net N$2: track 113.8 -> 118.8 mm
- net GND: track 0.00 -> 2.40 mm
- net N$20: track 73.9 -> 75.7 mm
- net N$18: track 10.7 -> 12.2 mm
