File: TMK-EURO-0.1.1.sch (EAGLE design)
At the start: 56 parts, among them IC1 TL082P, U1 IN, U2 IN, U3 IN, U4 IN, U5 IN, U6 IN, U7 THONKICONNOLD

Commit message: final design frontpanel include
Parts:
- C11: device rcl:C-EU050-035X075 -> adafruit:C-US050-075X075
Changed lines of the file:
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@@
 <part name="U1" library="MusicThingModular" deviceset="THONKICONN" device="OLD" value="IN"/>
 <part name="S1" library="momentswitchREDlveewrergalmoer" deviceset="SPDT" device="PADS"/>
-<part name="C11" library="rcl" deviceset="C-EU" device="050-035X075" value="1uF"/>
+<part name="C11" library="adafruit" deviceset="C-US" device="050-075X075" value="1uF"/>
 <part name="VR13" library="MusicThingModular" deviceset="9MM_SNAP-IN_POT" device="_" value="250K"/>
 <part name="R14" library="adafruit" deviceset="R-US_" device="0207/7" value="100k"/>
@@
 </segment>
 </net>
-<net name="N$35" class="0">
+<net name="N$35" class="2">
 <segment>
 <pinref part="C9" gate="G$1" pin="2"/>
