File: TMK-EURO-0.1.1x.brd (EAGLE design)
At the start: 100 x 80 mm, 47 parts, among them IC1 TL082P, U1 TL072_, U2 IN, U3 TL072_, U5 IN, U6 IN, U7 THONKICONNOLD, X1 057-010-1

Commit message: Ready for breadboard v2
Parts:
- removed C10, C9: 100nF, rcl:C050-035X075
- removed R13: 47k, adafruit:0207/7
- removed R14: 100k, adafruit:0207/7
- removed U5, U6: IN, MusicThingModular:THONKICONN
- removed VR12: 500k, MusicThingModular:9MM_SNAP-IN_POT
- removed VR13: 250K, MusicThingModular:9MM_SNAP-IN_POT
Connections:
- removed net N$10: IC1.1, LED1.A, LED2.K, U1.5, VR10.2, VR10.3
- removed net N$16: R14.1, VR13.3
- removed net N$17: R14.2, U1.6, U1.7
- removed net N$25: C10.2, U6.P$3_TIP
- removed net N$27: R13.2, U3.1, U3.2
- removed net N$35: C9.2, U5.P$3_TIP
- removed net N$4: R13.1, VR12.3
- removed net OUTPUT1: C10.1, VR13.1, VR13.2
- removed net OUTPUT2: C9.1, VR12.1, VR12.2
- new net N$30: IC1.1, LED1.A, LED2.K, VR10.2, VR10.3
- net GND: no longer U5.P$1_SLEEVE, U6.P$1_SLEEVE
- net N$13: no longer U3.3
Changed lines of the file:
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@@
 <elements>
 <element name="C1" library="adafruit" package="E2-5" value="10uF" x="-54.61" y="59.69"/>
-<element name="C10" library="rcl" library_urn="urn:adsk.eagle:library:334" package="C050-035X075" value="100nF" x="-34.29" y="60.96"/>
 <element name="C11" library="adafruit" package="C050-075X075" value="1uF" x="-41.91" y="46.99"/>
 <element name="C2" library="rcl" library_urn="urn:adsk.eagle:library:334" package="C050-035X075" value="100nF" x="-59.69" y="46.99"/>
@@
 <element name="C6" library="adafruit" package="C050-030X075" value="2.2uF" x="-43.18" y="60.96"/>
 <element name="C7" library="gm-caps-electro-pol" package="080_035" value="100uF" x="-50.8" y="46.99"/>
-<element name="C9" library="rcl" library_urn="urn:adsk.eagle:library:334" package="C050-035X075" value="100nF" x="-25.4" y="60.96"/>
 <element name="D1" library="MusicThingModular" package="DO35-7" value="1N4148" x="-58.42" y="71.12"/>
 <element name="D3" library="MusicThingModular" package="DO35-7" value="1N4148" x="-68.58" y="71.12"/>
@@
 <element name="R11" library="adafruit" package="0207/7" value="10K" x="-17.78" y="71.12"/>
 <element name="R12" library="adafruit" package="0207/7" value="10K" x="-27.94" y="71.12"/>
-<element name="R13" library="adafruit" package="0207/7" value="47k" x="-38.1" y="71.12"/>
-<element name="R14" library="adafruit" package="0207/7" value="100k" x="-48.26" y="71.12"/>
 <element name="R3" library="adafruit" package="0207/7" value="100K" x="-29.21" y="66.04"/>
 <element name="R4" library="adafruit" package="0207/7" value="470" x="-39.37" y="66.04"/>
@@
 <element name="R8" library="adafruit" package="0207/7" value="10K" x="-69.85" y="66.04"/>
 <element name="U2" library="MusicThingModular" package="THONKICONN" value="IN" x="-39.37" y="7.62"/>
-<element name="U5" library="MusicThingModular" package="THONKICONN" value="IN" x="-49.53" y="7.62"/>
-<element name="U6" library="MusicThingModular" package="THONKICONN" value="IN" x="-59.69" y="7.62"/>
 <element name="U7" library="MusicThingModular" package="THONKICONN" value="THONKICONNOLD" x="-69.85" y="7.62"/>
 <element name="VR1" library="MusicThingModular" package="9MM_SNAP-IN_POT" value="100K" x="-19.05" y="22.86"/>
 <element name="VR10" library="MusicThingModular" package="9MM_SNAP-IN_POT" value="250K" x="-31.75" y="36.83"/>
-<element name="VR12" library="MusicThingModular" package="9MM_SNAP-IN_POT" value="500k" x="-44.45" y="36.83"/>
-<element name="VR13" library="MusicThingModular" package="9MM_SNAP-IN_POT" value="250K" x="-57.15" y="36.83"/>
 <element name="VR14" library="MusicThingModular" package="9MM_SNAP-IN_POT" value="10K" x="-69.85" y="36.83"/>
 <element name="VR16" library="MusicThingModular" package="9MM_SNAP-IN_POT" value="500K" x="-19.05" y="50.8"/>
@@
 <contactref element="U7" pad="P$1_SLEEVE"/>
 <contactref element="VR3" pad="1"/>
-<contactref element="U6" pad="P$1_SLEEVE"/>
-<contactref element="U5" pad="P$1_SLEEVE"/>
 <contactref element="C7" pad="-"/>
 <contactref element="X1" pad="4"/>
@@
 <contactref element="C3" pad="+"/>
 <wire x1="-69.85" y1="1.14" x2="-83.03" y2="-72.39" width="0" layer="19" extent="1-1"/>
-<wire x1="-59.69" y1="1.14" x2="-69.85" y2="1.14" width="0" layer="19" extent="1-1"/>
-<wire x1="-49.53" y1="1.14" x2="-59.69" y2="1.14" width="0" layer="19" extent="1-1"/>
-<wire x1="-39.37" y1="1.14" x2="-49.53" y2="1.14" width="0" layer="19" extent="1-1"/>
-<wire x1="-26.67" y1="6.35" x2="-39.37" y2="1.14" width="0" layer="19" extent="1-1"/>
-<wire x1="-26.67" y1="8.89" x2="-26.67" y2="6.35" width="0" layer="19" extent="1-1"/>
+<wire x1="-46.95" y1="15.86" x2="-69.85" y2="1.14" width="0" layer="19" extent="1-1"/>
+<wire x1="-34.25" y1="15.86" x2="-46.95" y2="15.86" width="0" layer="19" extent="1-1"/>
+<wire x1="-26.67" y1="8.89" x2="-34.25" y2="15.86" width="0" layer="19" extent="1-1"/>
+<wire x1="-26.67" y1="6.35" x2="-26.67" y2="8.89" width="0" layer="19" extent="1-1"/>
 <wire x1="-24.13" y1="6.35" x2="-26.67" y2="6.35" width="0" layer="19" extent="1-1"/>
 <wire x1="-24.13" y1="8.89" x2="-26.67" y2="8.89" width="0" layer="19" extent="1-1"/>
@@
 <wire x1="-21.59" y1="8.89" x2="-24.13" y2="8.89" width="0" layer="19" extent="1-1"/>
 <wire x1="-21.55" y1="15.86" x2="-21.59" y2="8.89" width="0" layer="19" extent="1-1"/>
-<wire x1="-34.25" y1="15.86" x2="-26.67" y2="8.89" width="0" layer="19" extent="1-1"/>
-<wire x1="-46.95" y1="15.86" x2="-34.25" y2="15.86" width="0" layer="19" extent="1-1"/>
+<wire x1="-39.37" y1="1.14" x2="-26.67" y2="6.35" width="0" layer="19" extent="1-1"/>
 <wire x1="-21.55" y1="29.83" x2="-21.55" y2="15.86" width="0" layer="19" extent="1-1"/>
 <wire x1="-19.05" y1="29.83" x2="-21.55" y2="29.83" width="0" layer="19" extent="1-1"/>
@@
 <wire x1="-21.59" y1="71.12" x2="-22.86" y2="67.31" width="0" layer="19" extent="1-1"/>
 </signal>
-<signal name="N$10" class="2">
-<contactref element="VR10" pad="2"/>
-<contactref element="IC1" pad="1"/>
-<contactref element="LED1" pad="A"/>
-<contactref element="LED2" pad="K"/>
-<contactref element="VR10" pad="3"/>
-<contactref element="U1" pad="5"/>
-<wire x1="-31.75" y1="29.83" x2="-74.93" y2="-16.51" width="0" layer="19" extent="1-1"/>
-<wire x1="-29.25" y1="29.83" x2="-31.75" y2="29.83" width="0" layer="19" extent="1-1"/>
-<wire x1="-34.29" y1="44.45" x2="-31.75" y2="29.83" width="0" layer="19" extent="1-1"/>
-<wire x1="-20.32" y1="67.31" x2="-34.29" y2="44.45" width="0" layer="19" extent="1-1"/>
-<wire x1="-67.31" y1="59.69" x2="-34.29" y2="44.45" width="0" layer="19" extent="1-1"/>
-</signal>
 <signal name="N$6" class="2">
 <contactref element="R7" pad="2"/>
@@
 <contactref element="R12" pad="2"/>
 <contactref element="D1" pad="C"/>
-<contactref element="U3" pad="3"/>
-<wire x1="-67.35" y1="29.83" x2="-77.47" y2="-45.72" width="0" layer="19" extent="1-1"/>
-<wire x1="-62.23" y1="71.12" x2="-67.35" y2="29.83" width="0" layer="19" extent="1-1"/>
-<wire x1="-24.13" y1="71.12" x2="-62.23" y2="71.12" width="0" layer="19" extent="1-1"/>
+<wire x1="-62.23" y1="71.12" x2="-24.13" y2="71.12" width="0" layer="19" extent="1-1"/>
+<wire x1="-67.35" y1="29.83" x2="-62.23" y2="71.12" width="0" layer="19" extent="1-1"/>
 </signal>
 <signal name="N$14">
@@
 <wire x1="-16.55" y1="29.83" x2="-40.64" y2="60.96" width="0" layer="19" extent="1-1"/>
 </signal>
-<signal name="OUTPUT1" class="2">
-<contactref element="VR13" pad="2"/>
-<contactref element="C10" pad="1"/>
-<contactref element="VR13" pad="1"/>
-<wire x1="-57.15" y1="29.83" x2="-59.65" y2="29.83" width="0" layer="19" extent="1-1"/>
-<wire x1="-36.83" y1="60.96" x2="-57.15" y2="29.83" width="0" layer="19" extent="1-1"/>
-</signal>
-<signal name="N$25" class="2">
-<contactref element="C10" pad="2"/>
-<contactref element="U6" pad="P$3_TIP"/>
-<wire x1="-31.75" y1="60.96" x2="-59.69" y2="12.46" width="0" layer="19" extent="1-1"/>
-</signal>
-<signal name="OUTPUT2">
-<contactref element="VR12" pad="2"/>
-<contactref element="C9" pad="1"/>
-<contactref element="VR12" pad="1"/>
-<wire x1="-44.45" y1="29.83" x2="-27.94" y2="60.96" width="0" layer="19" extent="1-1"/>
-<wire x1="-46.95" y1="29.83" x2="-44.45" y2="29.83" width="0" layer="19" extent="1-1"/>
-</signal>
-<signal name="N$35" class="2">
-<contactref element="C9" pad="2"/>
-<contactref element="U5" pad="P$3_TIP"/>
-<wire x1="-49.53" y1="12.46" x2="-22.86" y2="60.96" width="0" layer="19" extent="1-1"/>
-</signal>
 <signal name="N$38">
 <contactref element="X1" pad="9"/>
@@
 <wire x1="-19.05" y1="6.35" x2="-19.05" y2="8.89" width="0" layer="19" extent="1-1"/>
 </signal>
-<signal name="N$16">
-<contactref element="R14" pad="1"/>
-<contactref element="VR13" pad="3"/>
-<wire x1="-52.07" y1="71.12" x2="-54.65" y2="29.83" width="0" layer="19" extent="1-1"/>
-</signal>
 <signal name="N$26" class="2">
 <contactref element="IC1" pad="3"/>
@@
 <wire x1="-66.04" y1="46.99" x2="-59.65" y2="15.86" width="0" layer="19" extent="1-1"/>
 <wire x1="-29.21" y1="44.45" x2="-66.04" y2="46.99" width="0" layer="19" extent="1-1"/>
-</signal>
-<signal name="N$4">
-<contactref element="R13" pad="1"/>
-<contactref element="VR12" pad="3"/>
-<wire x1="-41.95" y1="29.83" x2="-41.91" y2="71.12" width="0" layer="19" extent="1-1"/>
 </signal>
 <signal name="N$15">
@@
 <wire x1="-74.93" y1="-24.13" x2="-74.93" y2="-45.72" width="0" layer="19" extent="1-1"/>
 </signal>
-<signal name="N$17">
-<contactref element="U1" pad="7"/>
-<contactref element="R14" pad="2"/>
-<contactref element="U1" pad="6"/>
-<wire x1="-77.47" y1="-16.51" x2="-80.01" y2="-16.51" width="0" layer="19" extent="1-1"/>
-<wire x1="-44.45" y1="71.12" x2="-77.47" y2="-16.51" width="0" layer="19" extent="1-1"/>
-</signal>
-<signal name="N$27">
-<contactref element="U3" pad="1"/>
-<contactref element="U3" pad="2"/>
-<contactref element="R13" pad="2"/>
-<wire x1="-80.01" y1="-45.72" x2="-82.55" y2="-45.72" width="0" layer="19" extent="1-1"/>
-<wire x1="-34.29" y1="71.12" x2="-80.01" y2="-45.72" width="0" layer="19" extent="1-1"/>
-</signal>
 <signal name="N$28">
 <contactref element="U3" pad="7"/>
@@
 <wire x1="-19.05" y1="43.8" x2="-74.93" y2="-38.1" width="0" layer="19" extent="1-1"/>
 </signal>
+<signal name="N$30" class="2">
+<contactref element="VR10" pad="2"/>
+<contactref element="IC1" pad="1"/>
+<contactref element="LED1" pad="A"/>
+<contactref element="LED2" pad="K"/>
+<contactref element="VR10" pad="3"/>
+<wire x1="-34.29" y1="44.45" x2="-20.32" y2="67.31" width="0" layer="19" extent="1-1"/>
+<wire x1="-31.75" y1="29.83" x2="-34.29" y2="44.45" width="0" layer="19" extent="1-1"/>
+<wire x1="-29.25" y1="29.83" x2="-31.75" y2="29.83" width="0" layer="19" extent="1-1"/>
+<wire x1="-67.31" y1="59.69" x2="-34.29" y2="44.45" width="0" layer="19" extent="1-1"/>
+</signal>
 </signals>

Commit message: Ground switch input jack
Normal to groudn on input switch
Connections:
- removed net N$1: U2.P$2_SWITCH
- net GND: now also U2.P$2_SWITCH
Changed lines of the file:
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@@
 <?xml version="1.0" encoding="utf-8"?>
 <!DOCTYPE eagle SYSTEM "eagle.dtd">
-<eagle version="8.2.2">
+<eagle version="7.6.0">
 <drawing>
 <settings>
@@
 <element name="C1" library="adafruit" package="E2-5" value="10uF" x="-54.61" y="59.69"/>
 <element name="C11" library="adafruit" package="C050-075X075" value="1uF" x="-41.91" y="46.99"/>
-<element name="C2" library="rcl" library_urn="urn:adsk.eagle:library:334" package="C050-035X075" value="100nF" x="-59.69" y="46.99"/>
-<element name="C4" library="rcl" library_urn="urn:adsk.eagle:library:334" package="C050-035X075" value="100nF" x="-68.58" y="46.99"/>
-<element name="C5" library="rcl" library_urn="urn:adsk.eagle:library:334" package="C050-035X075" value="100nF" x="-16.51" y="60.96"/>
+<element name="C2" library="rcl" package="C050-035X075" value="100nF" x="-59.69" y="46.99"/>
+<element name="C4" library="rcl" package="C050-035X075" value="100nF" x="-68.58" y="46.99"/>
+<element name="C5" library="rcl" package="C050-035X075" value="100nF" x="-16.51" y="60.96"/>
 <element name="C6" library="adafruit" package="C050-030X075" value="2.2uF" x="-43.18" y="60.96"/>
 <element name="C7" library="gm-caps-electro-pol" package="080_035" value="100uF" x="-50.8" y="46.99"/>
@@
 <element name="D6" library="MusicThingModular" package="DO35-7" value="1N4148" x="-38.1" y="76.2"/>
 <element name="D7" library="MusicThingModular" package="DO35-7" value="1N5817" x="-48.26" y="76.2"/>
-<element name="IC1" library="linear" library_urn="urn:adsk.eagle:library:262" package="DIL08" value="TL082P" x="-30.48" y="48.26">
+<element name="IC1" library="linear" package="DIL08" value="TL082P" x="-30.48" y="48.26">
 <attribute name="DATA_SHEET" value="&lt;a href=&quot;http://www.ti.com/lit/ds/symlink/tl084a.pdf&quot;&gt; Data sheet &lt;/a&gt;" x="-30.48" y="48.26" size="1.778" layer="27" display="off"/>
 </element>
@@
 <element name="VR8" library="MusicThingModular" package="9MM_SNAP-IN_POT" value="50K" x="-69.85" y="22.86"/>
 <element name="VR9" library="MusicThingModular" package="9MM_SNAP-IN_POT" value="10K" x="-19.05" y="36.83"/>
-<element name="X1" library="con-panduit" library_urn="urn:adsk.eagle:library:169" package="057-010-1" value="057-010-1" x="-24.13" y="7.62">
+<element name="X1" library="con-panduit" package="057-010-1" value="057-010-1" x="-24.13" y="7.62">
 <attribute name="MF" value="" x="-24.13" y="7.62" size="1.778" layer="27" display="off"/>
 <attribute name="MPN" value="" x="-24.13" y="7.62" size="1.778" layer="27" display="off"/>
@@
 <contactref element="U2" pad="P$3_TIP"/>
 <wire x1="-16.55" y1="15.86" x2="-39.37" y2="12.46" width="0" layer="19" extent="1-1"/>
-</signal>
-<signal name="N$1">
-<contactref element="U2" pad="P$2_SWITCH"/>
 </signal>
 <signal name="GND" class="1">
@@
 <contactref element="X1" pad="7"/>
 <contactref element="C3" pad="+"/>
+<contactref element="U2" pad="P$2_SWITCH"/>
 <wire x1="-69.85" y1="1.14" x2="-83.03" y2="-72.39" width="0" layer="19" extent="1-1"/>
 <wire x1="-46.95" y1="15.86" x2="-69.85" y2="1.14" width="0" layer="19" extent="1-1"/>
@@
 <wire x1="-21.59" y1="8.89" x2="-24.13" y2="8.89" width="0" layer="19" extent="1-1"/>
 <wire x1="-21.55" y1="15.86" x2="-21.59" y2="8.89" width="0" layer="19" extent="1-1"/>
-<wire x1="-39.37" y1="1.14" x2="-26.67" y2="6.35" width="0" layer="19" extent="1-1"/>
+<wire x1="-39.37" y1="4.24" x2="-34.25" y2="15.86" width="0" layer="19" extent="1-1"/>
+<wire x1="-39.37" y1="1.14" x2="-39.37" y2="4.24" width="0" layer="19" extent="1-1"/>
 <wire x1="-21.55" y1="29.83" x2="-21.55" y2="15.86" width="0" layer="19" extent="1-1"/>
 <wire x1="-19.05" y1="29.83" x2="-21.55" y2="29.83" width="0" layer="19" extent="1-1"/>
@@
 </board>
 </drawing>
-<compatibility>
-<note version="8.2" severity="warning">
-Since Version 8.2, Eagle supports online libraries. The ids
-of those online libraries will not be understood (or retained)
-with this version.
-</note>
-</compatibility>
 </eagle>
