File: TMK-EURO-0.1.1x.brd (EAGLE design)
At the start: 100 x 80 mm, 39 parts, among them IC1 TL082P, U1 TL072_, U2 IN, U3 TL072_, U7 THONKICONNOLD, X1 057-010-1

Commit message: Buffered Euro Friendly
Ready for tewaking and CV-inputs?
Parts:
- removed C1: 10uF, adafruit:E2-5
- removed R3, R5: 100K, adafruit:0207/7
- removed VR3: 1k, MusicThingModular:9MM_SNAP-IN_POT
- C11: value 1uF -> 4.7uF
- IC1: value TL082P -> TL072
Connections:
- removed net N$23: R3.1, VR3.2
- removed net VR: C1.+, IC1.5, R3.2, R5.1, R7.1, R8.2
- net +12V: no longer VR3.3
- net GND: now also IC1.5, R7.1; no longer C1.-, R5.2, VR3.1
- net N$26: no longer VR7.1
- net N$28: now also U1.6, U1.7; no longer U3.6, U3.7
- net N$29: now also U1.5; no longer U3.5
- net N$7: now also VR7.1
- net N$8: now also R8.2
Changed lines of the file:
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@@
 <?xml version="1.0" encoding="utf-8"?>
 <!DOCTYPE eagle SYSTEM "eagle.dtd">
-<eagle version="7.6.0">
+<eagle version="8.3.2">
 <drawing>
 <settings>
 <setting alwaysvectorfont="yes"/>
+<setting keepoldvectorfont="yes"/>
 <setting verticaltext="up"/>
 </settings>
@@
 </autorouter>
 <elements>
-<element name="C1" library="adafruit" package="E2-5" value="10uF" x="-54.61" y="59.69"/>
-<element name="C11" library="adafruit" package="C050-075X075" value="1uF" x="-41.91" y="46.99"/>
+<element name="C11" library="adafruit" package="C050-075X075" value="4.7uF" x="-41.91" y="46.99"/>
 <element name="C2" library="rcl" package="C050-035X075" value="100nF" x="-59.69" y="46.99"/>
 <element name="C4" library="rcl" package="C050-035X075" value="100nF" x="-68.58" y="46.99"/>
@@
 <element name="D6" library="MusicThingModular" package="DO35-7" value="1N4148" x="-38.1" y="76.2"/>
 <element name="D7" library="MusicThingModular" package="DO35-7" value="1N5817" x="-48.26" y="76.2"/>
-<element name="IC1" library="linear" package="DIL08" value="TL082P" x="-30.48" y="48.26">
+<element name="IC1" library="linear" package="DIL08" value="TL072" x="-30.48" y="48.26">
 <attribute name="DATA_SHEET" value="&lt;a href=&quot;http://www.ti.com/lit/ds/symlink/tl084a.pdf&quot;&gt; Data sheet &lt;/a&gt;" x="-30.48" y="48.26" size="1.778" layer="27" display="off"/>
 </element>
@@
 <element name="R11" library="adafruit" package="0207/7" value="10K" x="-17.78" y="71.12"/>
 <element name="R12" library="adafruit" package="0207/7" value="10K" x="-27.94" y="71.12"/>
-<element name="R3" library="adafruit" package="0207/7" value="100K" x="-29.21" y="66.04"/>
 <element name="R4" library="adafruit" package="0207/7" value="470" x="-39.37" y="66.04"/>
-<element name="R5" library="adafruit" package="0207/7" value="100K" x="-49.53" y="66.04"/>
 <element name="R7" library="adafruit" package="0207/7" value="1K" x="-59.69" y="66.04"/>
 <element name="R8" library="adafruit" package="0207/7" value="10K" x="-69.85" y="66.04"/>
@@
 <element name="VR16" library="MusicThingModular" package="9MM_SNAP-IN_POT" value="500K" x="-19.05" y="50.8"/>
 <element name="VR2" library="MusicThingModular" package="9MM_SNAP-IN_POT" value="500K" x="-31.75" y="22.86"/>
-<element name="VR3" library="MusicThingModular" package="9MM_SNAP-IN_POT" value="1k" x="-44.45" y="22.86"/>
 <element name="VR7" library="MusicThingModular" package="9MM_SNAP-IN_POT" value="250K" x="-57.15" y="22.86"/>
 <element name="VR8" library="MusicThingModular" package="9MM_SNAP-IN_POT" value="50K" x="-69.85" y="22.86"/>
@@
 <contactref element="VR9" pad="1"/>
 <contactref element="VR9" pad="2"/>
-<contactref element="R5" pad="2"/>
-<contactref element="C1" pad="-"/>
 <contactref element="IC1" pad="4"/>
 <contactref element="D6" pad="C"/>
@@
 <contactref element="VR16" pad="1"/>
 <contactref element="U7" pad="P$1_SLEEVE"/>
-<contactref element="VR3" pad="1"/>
 <contactref element="C7" pad="-"/>
 <contactref element="X1" pad="4"/>
@@
 <contactref element="C3" pad="+"/>
 <contactref element="U2" pad="P$2_SWITCH"/>
+<contactref element="R7" pad="1"/>
+<contactref element="IC1" pad="5"/>
 <wire x1="-69.85" y1="1.14" x2="-83.03" y2="-72.39" width="0" layer="19" extent="1-1"/>
-<wire x1="-46.95" y1="15.86" x2="-69.85" y2="1.14" width="0" layer="19" extent="1-1"/>
-<wire x1="-34.25" y1="15.86" x2="-46.95" y2="15.86" width="0" layer="19" extent="1-1"/>
+<wire x1="-39.37" y1="1.14" x2="-69.85" y2="1.14" width="0" layer="19" extent="1-1"/>
+<wire x1="-39.37" y1="4.24" x2="-39.37" y2="1.14" width="0" layer="19" extent="1-1"/>
+<wire x1="-34.25" y1="15.86" x2="-39.37" y2="4.24" width="0" layer="19" extent="1-1"/>
 <wire x1="-26.67" y1="8.89" x2="-34.25" y2="15.86" width="0" layer="19" extent="1-1"/>
 <wire x1="-26.67" y1="6.35" x2="-26.67" y2="8.89" width="0" layer="19" extent="1-1"/>
@@
 <wire x1="-21.59" y1="8.89" x2="-24.13" y2="8.89" width="0" layer="19" extent="1-1"/>
 <wire x1="-21.55" y1="15.86" x2="-21.59" y2="8.89" width="0" layer="19" extent="1-1"/>
-<wire x1="-39.37" y1="4.24" x2="-34.25" y2="15.86" width="0" layer="19" extent="1-1"/>
-<wire x1="-39.37" y1="1.14" x2="-39.37" y2="4.24" width="0" layer="19" extent="1-1"/>
 <wire x1="-21.55" y1="29.83" x2="-21.55" y2="15.86" width="0" layer="19" extent="1-1"/>
 <wire x1="-19.05" y1="29.83" x2="-21.55" y2="29.83" width="0" layer="19" extent="1-1"/>
 <wire x1="-21.55" y1="43.8" x2="-21.55" y2="29.83" width="0" layer="19" extent="1-1"/>
 <wire x1="-26.67" y1="44.45" x2="-21.55" y2="43.8" width="0" layer="19" extent="1-1"/>
-<wire x1="-13.97" y1="60.96" x2="-21.55" y2="43.8" width="0" layer="19" extent="1-1"/>
+<wire x1="-26.67" y1="52.07" x2="-26.67" y2="44.45" width="0" layer="19" extent="1-1"/>
+<wire x1="-13.97" y1="60.96" x2="-26.67" y2="52.07" width="0" layer="19" extent="1-1"/>
 <wire x1="-49.05" y1="46.99" x2="-26.67" y2="44.45" width="0" layer="19" extent="1-1"/>
-<wire x1="-53.594" y1="59.69" x2="-49.05" y2="46.99" width="0" layer="19" extent="1-1"/>
-<wire x1="-45.72" y1="66.04" x2="-53.594" y2="59.69" width="0" layer="19" extent="1-1"/>
-<wire x1="-41.91" y1="76.2" x2="-45.72" y2="66.04" width="0" layer="19" extent="1-1"/>
-<wire x1="-64.77" y1="71.12" x2="-53.594" y2="59.69" width="0" layer="19" extent="1-1"/>
+<wire x1="-63.5" y1="66.04" x2="-49.05" y2="46.99" width="0" layer="19" extent="1-1"/>
+<wire x1="-64.77" y1="71.12" x2="-63.5" y2="66.04" width="0" layer="19" extent="1-1"/>
+<wire x1="-41.91" y1="76.2" x2="-64.77" y2="71.12" width="0" layer="19" extent="1-1"/>
 </signal>
 <signal name="N$3" class="2">
@@
 <wire x1="-54.65" y1="15.86" x2="-57.15" y2="15.86" width="0" layer="19" extent="1-1"/>
 <wire x1="-73.66" y1="66.04" x2="-57.15" y2="15.86" width="0" layer="19" extent="1-1"/>
-</signal>
-<signal name="VR" class="1">
-<contactref element="R8" pad="2"/>
-<contactref element="R7" pad="1"/>
-<contactref element="IC1" pad="5"/>
-<contactref element="R3" pad="2"/>
-<contactref element="R5" pad="1"/>
-<contactref element="C1" pad="+"/>
-<wire x1="-26.67" y1="52.07" x2="-25.4" y2="66.04" width="0" layer="19" extent="1-1"/>
-<wire x1="-53.34" y1="66.04" x2="-25.4" y2="66.04" width="0" layer="19" extent="1-1"/>
-<wire x1="-55.626" y1="59.69" x2="-53.34" y2="66.04" width="0" layer="19" extent="1-1"/>
-<wire x1="-63.5" y1="66.04" x2="-55.626" y2="59.69" width="0" layer="19" extent="1-1"/>
-<wire x1="-66.04" y1="66.04" x2="-63.5" y2="66.04" width="0" layer="19" extent="1-1"/>
 </signal>
 <signal name="N$7" class="1">
@@
 <contactref element="VR8" pad="1"/>
 <contactref element="VR10" pad="1"/>
+<contactref element="VR7" pad="1"/>
+<wire x1="-59.65" y1="15.86" x2="-72.35" y2="15.86" width="0" layer="19" extent="1-1"/>
 <wire x1="-72.35" y1="29.83" x2="-72.35" y2="15.86" width="0" layer="19" extent="1-1"/>
+<wire x1="-34.25" y1="29.83" x2="-59.65" y2="15.86" width="0" layer="19" extent="1-1"/>
 <wire x1="-64.77" y1="59.69" x2="-72.35" y2="29.83" width="0" layer="19" extent="1-1"/>
-<wire x1="-34.25" y1="29.83" x2="-72.35" y2="29.83" width="0" layer="19" extent="1-1"/>
 <wire x1="-22.86" y1="67.31" x2="-34.25" y2="29.83" width="0" layer="19" extent="1-1"/>
 <wire x1="-21.59" y1="71.12" x2="-22.86" y2="67.31" width="0" layer="19" extent="1-1"/>
@@
 </signal>
 <signal name="+12V" class="1">
-<contactref element="VR3" pad="3"/>
 <contactref element="D7" pad="C"/>
 <contactref element="C7" pad="+"/>
@@
 <contactref element="U3" pad="8"/>
 <wire x1="-82.55" y1="-16.51" x2="-82.55" y2="-38.1" width="0" layer="19" extent="1-1"/>
-<wire x1="-41.95" y1="15.86" x2="-82.55" y2="-16.51" width="0" layer="19" extent="1-1"/>
-<wire x1="-52.55" y1="46.99" x2="-41.95" y2="15.86" width="0" layer="19" extent="1-1"/>
+<wire x1="-52.55" y1="46.99" x2="-82.55" y2="-16.51" width="0" layer="19" extent="1-1"/>
 <wire x1="-34.29" y1="52.07" x2="-52.55" y2="46.99" width="0" layer="19" extent="1-1"/>
 <wire x1="-52.07" y1="76.2" x2="-52.55" y2="46.99" width="0" layer="19" extent="1-1"/>
@@
 <contactref element="U7" pad="P$2_SWITCH"/>
 </signal>
-<signal name="N$23" class="1">
-<contactref element="VR3" pad="2"/>
-<contactref element="R3" pad="1"/>
-<wire x1="-44.45" y1="15.86" x2="-33.02" y2="66.04" width="0" layer="19" extent="1-1"/>
-</signal>
 <signal name="N$8">
 <contactref element="VR9" pad="3"/>
 <contactref element="C6" pad="2"/>
+<contactref element="R8" pad="2"/>
+<wire x1="-66.04" y1="66.04" x2="-40.64" y2="60.96" width="0" layer="19" extent="1-1"/>
 <wire x1="-16.55" y1="29.83" x2="-40.64" y2="60.96" width="0" layer="19" extent="1-1"/>
 </signal>
@@
 <signal name="N$26" class="2">
 <contactref element="IC1" pad="3"/>
-<contactref element="VR7" pad="1"/>
 <contactref element="C4" pad="2"/>
-<wire x1="-66.04" y1="46.99" x2="-59.65" y2="15.86" width="0" layer="19" extent="1-1"/>
 <wire x1="-29.21" y1="44.45" x2="-66.04" y2="46.99" width="0" layer="19" extent="1-1"/>
 </signal>
@@
 </signal>
 <signal name="N$28">
-<contactref element="U3" pad="7"/>
-<contactref element="U3" pad="6"/>
 <contactref element="U7" pad="P$3_TIP"/>
-<wire x1="-77.47" y1="-38.1" x2="-80.01" y2="-38.1" width="0" layer="19" extent="1-1"/>
-<wire x1="-69.85" y1="12.46" x2="-77.47" y2="-38.1" width="0" layer="19" extent="1-1"/>
+<contactref element="U1" pad="6"/>
+<contactref element="U1" pad="7"/>
+<wire x1="-77.47" y1="-16.51" x2="-80.01" y2="-16.51" width="0" layer="19" extent="1-1"/>
+<wire x1="-69.85" y1="12.46" x2="-77.47" y2="-16.51" width="0" layer="19" extent="1-1"/>
 </signal>
 <signal name="N$29">
 <contactref element="VR16" pad="2"/>
-<contactref element="U3" pad="5"/>
-<wire x1="-19.05" y1="43.8" x2="-74.93" y2="-38.1" width="0" layer="19" extent="1-1"/>
+<contactref element="U1" pad="5"/>
+<wire x1="-19.05" y1="43.8" x2="-74.93" y2="-16.51" width="0" layer="19" extent="1-1"/>
 </signal>
 <signal name="N$30" class="2">

Commit message: FinalCleanUp
Ready for testing, adding CV
Parts:
- removed D4, D5, D6: 1N4148, MusicThingModular:DO35-7
- removed R8: 10K, adafruit:0207/7
- removed U3: TL072_, EURACK-MASTER-LIB:DIL08
- removed VR10, VR7: 250K, MusicThingModular:9MM_SNAP-IN_POT
- added C1, C10, C8, C9: 100nF, rcl:C050-035X075
- added R1: 100K, EURACK-MASTER-LIB:7MM_RESISTOR
- added R2: 10K, adafruit:0207/7
- C2: value 100nF -> 56pF
- VR1: value 100K -> 250K
- moved D3 240.2 mm to (-78.7, -168.9)
Connections:
- removed net N$21: D4.C, D5.A
- removed net N$22: D5.C, D6.A
- new net N$1: R1.1, VR1.2
- new net N$10: C1.2, C10.1
- new net N$4: R1.2, U1.3
- net +12V: now also C1.1, C8.1; no longer U3.8
- net -12V: now also C10.2, C9.2, IC1.4; no longer U3.4
- net GND: no longer D6.C, IC1.4
- net N$15: now also R2.2, U7.P$3_TIP; no longer U1.3, VR1.2
- net N$20: no longer D4.A
- net N$28: now also R2.1; no longer U7.P$3_TIP
- net N$30: no longer VR10.2, VR10.3
- net N$5: now also C8.2, C9.1; no longer R8.1, VR7.2, VR7.3
- net N$7: no longer VR10.1, VR7.1
- net N$8: no longer R8.2
